File: hardware/pcb/mcu.kicad_sch (KiCad schematic)
At the start: 15 parts, among them SW201 SKRHAAE010, SW202 SKRPABE010, SW203 SKRPABE010, SW204 SKRPABE010, SW205 SKRPABE010, SW206 SKRPABE010, U202 74AHCT125BQ,115, U203 MIC5219-3.3YM5, U402 ESP32-S3-MINI-1-N8

Commit message: forgot journal
Parts:
- added C207: 0.1uF, Capacitor_SMD:C_0603_1608Metric, symbol PCM_Capacitor_AKL:C_0603
- added J201, J202: Conn_01x04_MountingPin, Connector_JST:JST_GH_SM04B-GHS-TB_1x04-1MP_P1.25mm_Horizontal, symbol Connector_Generic_MountingPin:Conn_01x04_MountingPin
- added SW207: SKRPABE010, easyeda2kicad:KEY-SMD_4P-L4.2-W3.2-P2.20-LS4.6, symbol easyeda2kicad:SKRPABE010
Connections:
- net GND: now also C207.1, J201.4 (Pin_4), J201.MP (MountPin), J202.4 (Pin_4), J202.MP (MountPin), SW207.4
- net Q1_I: now also U402.8 (IO4)
- net Q2_I: now also U402.9 (IO5)
- net Q3_I: now also U402.10 (IO6)
- net Q4_I: now also U402.11 (IO7)
- net D-: now reaches U402.23 (IO19)
- net D-: now also J201.1 (Pin_1)
- net D+: now reaches U402.24 (IO20)
- net D+: now also J201.2 (Pin_2)
- net TX: now reaches U402.39 (TXD0)
- net TX: now also J202.2 (Pin_2)
- net RX: now reaches U402.40 (RXD0)
- net RX: now also J202.1 (Pin_1)
- net EN: now reaches U402.41 (IO45)
- net EN: now also C207.2, SW207.1
- net 5V renamed 5V_BEC
- net 5V_BEC: now also J201.3 (Pin_3), J202.3 (Pin_3)
