File: hardware/pcb/pcb.kicad_pcb (KiCad board)
At the start: 2 copper layers, 141 parts, among them J401 USB_C_Receptacle_USB2.0_16P, SW201 SKRHAAE010, SW202 SKRPABE010, SW203 SKRPABE010, SW204 SKRPABE010, SW205 SKRPABE010, SW206 SKRPABE010, SW401 DSHP03TS-S, U202 74AHCT125BQ,115, U203 MIC5219-3.3YM5, U401 CH224K, U402 ESP32-S3-MINI-1-N8, U501 MP9943GQ

Commit message: forgot journal
Parts:
- added C207: 0.1uF, Capacitor_SMD:C_0603_1608Metric, F.Cu at (31.4, 67.5)
- added J201: Conn_01x04_MountingPin, Connector_JST:JST_GH_SM04B-GHS-TB_1x04-1MP_P1.25mm_Horizontal, B.Cu at (27.2, 63.2)
- added J202: Conn_01x04_MountingPin, Connector_JST:JST_GH_SM04B-GHS-TB_1x04-1MP_P1.25mm_Horizontal, B.Cu at (27.2, 53.8)
- added SW207: SKRPABE010, easyeda2kicad:KEY-SMD_4P-L4.2-W3.2-P2.20-LS4.6, F.Cu at (27.6, 67.5)
- C401, C501, C502, C503, C504, C505, C506, C507, J401, L501, LED401, R401, R402, R403, R404, R405, R406, R501, R502, R503, R504, R505, R506, SW401, U401, U501: moved to B.Cu
- moved C506 43.9 mm to (49.4, 51.1), turned to 180 degrees
- moved R504 43.8 mm to (46.7, 53.2), turned to -90 degrees
- moved C507 40.3 mm to (49.4, 53.7), turned to 180 degrees
- moved C401 38.9 mm to (56.4, 84.5), turned to -90 degrees
- moved R406 38.6 mm to (47.0, 84.3), turned to -90 degrees
- moved R404 38.6 mm to (43.7, 84.2), turned to -90 degrees
- moved R405 38.6 mm to (45.4, 84.2), turned to -90 degrees
- moved LED401 38.6 mm to (53.8, 84.2)
- moved R403 36.2 mm to (53.8, 82.3)
- moved L501 35.6 mm to (48.4, 58.1), turned to 90 degrees
- moved R402 33.4 mm to (54.6, 79.3), turned to 90 degrees
- moved J401 31.8 mm to (60.5, 77.3), turned to -90 degrees
- moved U401 31.7 mm to (51.1, 77.1), turned to 90 degrees
- moved SW401 31.6 mm to (45.4, 77.0)
- moved C504 30.8 mm to (53.1, 56.9), turned to 0 degrees
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Connections:
- C201 pad 1: 5V -> 5V_BEC
- C202 pad 1: 5V -> 5V_BEC
- C502 pad 1: Net-(U501-VIN) -> VBUS
- C503 pad 1: Net-(U501-VIN) -> VBUS
- C504 pad 1: Net-(U501-VIN) -> VBUS
- LED301 pad 4: 5V -> 5V_BEC
- LED302 pad 4: 5V -> 5V_BEC
- LED303 pad 4: unconnected-(LED303-VDD-Pad4) -> 5V_BEC
- LED304 pad 4: 5V -> 5V_BEC
- LED305 pad 4: 5V -> 5V_BEC
- LED306 pad 4: 5V -> 5V_BEC
- LED307 pad 4: 5V -> 5V_BEC
- LED308 pad 4: unconnected-(LED308-VDD-Pad4) -> 5V_BEC
- LED309 pad 4: 5V -> 5V_BEC
- LED310 pad 4: 5V -> 5V_BEC
- LED311 pad 4: 5V -> 5V_BEC
- LED312 pad 4: 5V -> 5V_BEC
- LED313 pad 4: unconnected-(LED313-VDD-Pad4) -> 5V_BEC
- LED314 pad 4: 5V -> 5V_BEC
- LED315 pad 4: 5V -> 5V_BEC
- LED316 pad 4: 5V -> 5V_BEC
- LED317 pad 4: 5V -> 5V_BEC
- LED318 pad 4: unconnected-(LED318-VDD-Pad4) -> 5V_BEC
- LED319 pad 4: 5V -> 5V_BEC
- LED320 pad 4: 5V -> 5V_BEC
- LED321 pad 4: 5V -> 5V_BEC
- LED322 pad 4: 5V -> 5V_BEC
- LED323 pad 4: unconnected-(LED323-VDD-Pad4) -> 5V_BEC
- LED324 pad 4: 5V -> 5V_BEC
- LED325 pad 4: 5V -> 5V_BEC
- LED326 pad 4: 5V -> 5V_BEC
- LED327 pad 4: 5V -> 5V_BEC
- LED328 pad 4: unconnected-(LED328-VDD-Pad4) -> 5V_BEC
- LED329 pad 4: 5V -> 5V_BEC
- LED330 pad 4: 5V -> 5V_BEC
- LED331 pad 4: 5V -> 5V_BEC
- LED332 pad 4: 5V -> 5V_BEC
- LED333 pad 4: unconnected-(LED333-VDD-Pad4) -> 5V_BEC
- LED334 pad 4: 5V -> 5V_BEC
- LED335 pad 4: 5V -> 5V_BEC
- LED336 pad 4: 5V -> 5V_BEC
- LED337 pad 4: 5V -> 5V_BEC
- LED338 pad 4: unconnected-(LED338-VDD-Pad4) -> 5V_BEC
- LED339 pad 4: 5V -> 5V_BEC
- LED340 pad 4: 5V -> 5V_BEC
- LED341 pad 4: 5V -> 5V_BEC
- LED342 pad 4: 5V -> 5V_BEC
- LED343 pad 4: unconnected-(LED343-VDD-Pad4) -> 5V_BEC
- LED344 pad 4: 5V -> 5V_BEC
- LED345 pad 4: 5V -> 5V_BEC
- LED346 pad 4: 5V -> 5V_BEC
- LED347 pad 4: 5V -> 5V_BEC
- LED348 pad 4: unconnected-(LED348-VDD-Pad4) -> 5V_BEC
- LED349 pad 4: 5V -> 5V_BEC
- LED350 pad 4: 5V -> 5V_BEC
- LED351 pad 4: 5V -> 5V_BEC
- LED352 pad 4: 5V -> 5V_BEC
- LED353 pad 4: unconnected-(LED353-VDD-Pad4) -> 5V_BEC
- LED354 pad 4: 5V -> 5V_BEC
- LED355 pad 4: 5V -> 5V_BEC
- LED356 pad 4: 5V -> 5V_BEC
- LED357 pad 4: 5V -> 5V_BEC
- LED358 pad 4: unconnected-(LED358-VDD-Pad4) -> 5V_BEC
- LED359 pad 4: 5V -> 5V_BEC
- LED360 pad 4: 5V -> 5V_BEC
- LED361 pad 4: 5V -> 5V_BEC
- LED362 pad 4: 5V -> 5V_BEC
- LED363 pad 4: unconnected-(LED363-VDD-Pad4) -> 5V_BEC
- LED364 pad 4: 5V -> 5V_BEC
- LED365 pad 4: 5V -> 5V_BEC
- LED366 pad 4: 5V -> 5V_BEC
- LED367 pad 4: 5V -> 5V_BEC
- LED368 pad 4: unconnected-(LED368-VDD-Pad4) -> 5V_BEC
- LED369 pad 4: 5V -> 5V_BEC
- LED370 pad 4: 5V -> 5V_BEC
- LED371 pad 4: 5V -> 5V_BEC
- LED372 pad 4: 5V -> 5V_BEC
- LED373 pad 4: unconnected-(LED373-VDD-Pad4) -> 5V_BEC
- LED374 pad 4: 5V -> 5V_BEC
- LED375 pad 4: 5V -> 5V_BEC
- LED376 pad 4: 5V -> 5V_BEC
- LED377 pad 4: 5V -> 5V_BEC
- LED378 pad 4: unconnected-(LED378-VDD-Pad4) -> 5V_BEC
- LED379 pad 4: 5V -> 5V_BEC
- LED380 pad 4: 5V -> 5V_BEC
- LED381 pad 4: 5V -> 5V_BEC
- LED382 pad 4: 5V -> 5V_BEC
- LED383 pad 4: unconnected-(LED383-VDD-Pad4) -> 5V_BEC
- LED384 pad 4: 5V -> 5V_BEC
- LED385 pad 4: 5V -> 5V_BEC
- LED386 pad 4: 5V -> 5V_BEC
- LED387 pad 4: 5V -> 5V_BEC
- LED388 pad 4: unconnected-(LED388-VDD-Pad4) -> 5V_BEC
- LED389 pad 4: 5V -> 5V_BEC
- LED390 pad 4: 5V -> 5V_BEC
- LED391 pad 4: 5V -> 5V_BEC
- LED392 pad 4: 5V -> 5V_BEC
- LED393 pad 4: unconnected-(LED393-VDD-Pad4) -> 5V_BEC
- LED394 pad 4: 5V -> 5V_BEC
- LED395 pad 4: 5V -> 5V_BEC
- LED396 pad 4: 5V -> 5V_BEC
- LED397 pad 4: 5V -> 5V_BEC
- LED398 pad 4: unconnected-(LED398-VDD-Pad4) -> 5V_BEC
- LED399 pad 4: 5V -> 5V_BEC
- LED400 pad 4: 5V -> 5V_BEC
- R502 pad 1: Net-(U501-VIN) -> VBUS
- U203 pad 1: 5V -> 5V_BEC
- U203 pad 3: 5V -> 5V_BEC
- U402 pad 10: unconnected-(U402-IO6-Pad10) -> Q3_I
- U402 pad 11: unconnected-(U402-IO7-Pad11) -> Q4_I
- U402 pad 23: unconnected-(U402-IO19-Pad23) -> D-
- U402 pad 24: unconnected-(U402-IO20-Pad24) -> D+
- U402 pad 39: unconnected-(U402-TXD0-Pad39) -> TX
- U402 pad 40: unconnected-(U402-RXD0-Pad40) -> RX
- U402 pad 41: unconnected-(U402-IO45-Pad41) -> EN
- U402 pad 8: unconnected-(U402-IO4-Pad8) -> Q1_I
- U402 pad 9: unconnected-(U402-IO5-Pad9) -> Q2_I
- U501 pad 7: Net-(U501-VIN) -> VBUS
Routing:
- net Q1: track 0.00 -> 58.7 mm, vias 0 -> 2
- net 5V_BEC: track 0.00 -> 55.7 mm, vias 0 -> 103
- net Q2: track 0.00 -> 54.3 mm, vias 0 -> 2
- net Q4: track 0.00 -> 51.6 mm, vias 0 -> 2
- net B1: track 0.00 -> 47.6 mm
- net B4: track 0.00 -> 47.2 mm
- net Q3: track 0.00 -> 43.0 mm, vias 0 -> 2
- net VBUS: track 0.00 -> 39.2 mm, vias 0 -> 60
- net B5: track 0.00 -> 38.6 mm
- net B2: track 0.00 -> 32.1 mm
- net A: track 0.00 -> 30.5 mm, vias 0 -> 2
- net B: track 0.00 -> 30.4 mm, vias 0 -> 2
- net 3.3V: track 0.00 -> 30.4 mm, vias 0 -> 5
- net B3: track 0.00 -> 30.4 mm
- net Net-(R504-Pad1): track 0.00 -> 27.1 mm
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- added copper zone on F.Cu, net 3.3V
- added copper zone on B.Cu, net 5V_BEC
- added copper zone on F.Cu, net 5V_BEC
- added copper zone on In2.Cu, net 5V_BEC
- added copper zone on B.Cu, net GND
- added copper zone on F.Cu, net GND
- added copper zone on In1.Cu, net GND
- added copper zone on In2.Cu, net GND
- added copper zone on B.Cu, net Net-(U501-SW)
- added copper zone on B.Cu, net VBUS
Other:
- board outline added: 40 x 69 mm
- copper layers 2 -> 4
