File: hardware/pcb/quadrant.kicad_sch (KiCad schematic)
At the start: 100 parts

Commit message: forgot journal
Connections:
- net 5V is gone; now on net 5V_BEC: LED301.4 (VDD), LED302.4 (VDD), LED304.4 (VDD), LED305.4 (VDD), LED306.4 (VDD), LED307.4 (VDD), LED309.4 (VDD), LED310.4 (VDD), LED311.4 (VDD), LED312.4 (VDD), LED314.4 (VDD), LED315.4 (VDD), LED316.4 (VDD), LED317.4 (VDD), LED319.4 (VDD), LED320.4 (VDD), LED321.4 (VDD), LED322.4 (VDD), LED324.4 (VDD), LED325.4 (VDD), LED326.4 (VDD), LED327.4 (VDD), LED329.4 (VDD), LED330.4 (VDD), LED331.4 (VDD), LED332.4 (VDD), LED334.4 (VDD), LED335.4 (VDD), LED336.4 (VDD), LED337.4 (VDD), LED339.4 (VDD), LED340.4 (VDD), LED341.4 (VDD), LED342.4 (VDD), LED344.4 (VDD), LED345.4 (VDD), LED346.4 (VDD), LED347.4 (VDD), LED349.4 (VDD), LED350.4 (VDD), LED351.4 (VDD), LED352.4 (VDD), LED354.4 (VDD), LED355.4 (VDD), LED356.4 (VDD), LED357.4 (VDD), LED359.4 (VDD), LED360.4 (VDD), LED361.4 (VDD), LED362.4 (VDD), LED364.4 (VDD), LED365.4 (VDD), LED366.4 (VDD), LED367.4 (VDD), LED369.4 (VDD), LED370.4 (VDD), LED371.4 (VDD), LED372.4 (VDD), LED374.4 (VDD), LED375.4 (VDD), LED376.4 (VDD), LED377.4 (VDD), LED379.4 (VDD), LED380.4 (VDD), LED381.4 (VDD), LED382.4 (VDD), LED384.4 (VDD), LED385.4 (VDD), LED386.4 (VDD), LED387.4 (VDD), LED389.4 (VDD), LED390.4 (VDD), LED391.4 (VDD), LED392.4 (VDD), LED394.4 (VDD), LED395.4 (VDD), LED396.4 (VDD), LED397.4 (VDD), LED399.4 (VDD), LED400.4 (VDD)
- net 5V_BEC: now reaches LED333.4 (VDD)
- net 5V_BEC: now also LED303.4 (VDD), LED308.4 (VDD), LED313.4 (VDD), LED318.4 (VDD), LED323.4 (VDD), LED328.4 (VDD), LED338.4 (VDD), LED343.4 (VDD), LED348.4 (VDD), LED353.4 (VDD), LED358.4 (VDD), LED363.4 (VDD), LED368.4 (VDD), LED373.4 (VDD), LED378.4 (VDD), LED383.4 (VDD), LED388.4 (VDD), LED393.4 (VDD), LED398.4 (VDD)
