File: hardware/pcb/step-down.kicad_sch (KiCad schematic)
At the start: 15 parts, among them U501 MP9943GQ

Commit message: forgot journal
Connections:
- net VBUS: now reaches C502.1, C503.1, C504.1, R502.1, U501.7 (VIN)
Changed lines of the file:
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@@
+		)
+	)
+	(global_label "VBUS"
+		(shape input)
+		(at 174.625 93.345 0)
+		(fields_autoplaced yes)
+		(effects
+			(font
+				(size 1.27 1.27)
+			)
+			(justify left)
+		)
+		(property "Intersheetrefs" "${INTERSHEET_REFS}"
+			(at 182.5088 93.345 0)
+			(effects
+				(font
+					(size 1.27 1.27)
+				)
+				(justify left)
+				(hide yes)
+			)
 		)
 	)
